File: PCB/keyboard.kicad_pcb (KiCad board)
At the start: 2 copper layers, 100 x 100 mm, 47 parts, among them J1 Conn_01x04, J2 Conn_01x04, SW1 SW_Push, SW10 SW_Push, SW11 SW_Push, SW12 SW_Push, SW13 SW_Push, SW14 SW_Push, SW15 SW_Push, SW16 SW_Push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

Commit message: files
Parts:
- D18, D20, D3, D4, D6, D8: moved to B.Cu
- moved D5 80.8 mm to (90.5, 82.4)
- moved D4 64.5 mm to (131.9, 100.0)
- moved D1 60.0 mm to (109.5, 106.4)
- moved D2 59.8 mm to (109.5, 92.4)
- moved D17 52.0 mm to (118.7, 61.2), turned to 0 degrees
- moved D11 48.7 mm to (128.5, 90.3)
- moved D10 38.7 mm to (128.5, 73.4)
- moved D12 28.4 mm to (147.8, 82.9), turned to -90 degrees
- moved D19 13.4 mm to (155.5, 81.0), turned to 0 degrees
Routing:
- net Net-(D4-A): track 96.7 -> 4.93 mm
- net Net-(D5-A): track 95.1 -> 8.92 mm
- net Net-(D2-A): track 81.5 -> 8.77 mm
- net Rotary1: track 4.38 -> 66.0 mm, vias 0 -> 2
- net Net-(D1-A): track 91.3 -> 30.0 mm
- net ROW0: track 288.9 -> 240.7 mm, vias 1 -> 2
- net Net-(D10-A): track 68.0 -> 27.4 mm
- net Net-(D11-A): track 52.3 -> 19.2 mm
- net Net-(D12-A): track 20.8 -> 48.8 mm
- net ROW1: track 187.5 -> 206.5 mm
- net ROW2: track 182.2 -> 199.2 mm, vias 4 -> 5
- net Net-(D19-A): track 9.68 -> 5.82 mm, vias 1 -> 0
